File: hardware/s1_mini.sch (KiCad schematic (older format))
At the start: 10 parts

Commit message: Annotate parts.
Parts:
- removed U?: AP2114H-3.3TRG1, SOT-23, symbol APE8865NL-33-HF-3
- added R5: 10K, Resistors_SMD:R_0805_HandSoldering, symbol R_Small
- added U1: AP2114H, TO_SOT_Packages_SMD:SOT-223, symbol AP2114H
- C1, C2: renamed from C?; footprint (none) -> Capacitors_SMD:C_0805_HandSoldering
- P1: renamed from P?; footprint (none) -> CrumpPrints:USB_Board_Edge
- R1, R2, R3, R4: renamed from R?; footprint (none) -> Resistors_SMD:R_0805_HandSoldering
- U2: renamed from U?; footprint (none) -> CrumpPrints:SM200
- gave numbers to parts that had none: 1
Connections:
- net +3V3: now also R5.1, U1.2 (VOUT)
- net +5V: now also U1.3 (VIN)
- net GND: now also U1.1 (GND)
- net SNAP_PB5_PWM_INT: now also U3.14 (D1)
- net SNAP_PB6_PWM_INT: now also U3.13 (D2)
- net SNAP_PE4_PWM_INT: now also U3.12 (D3)
- net SNAP_PE5_PWM_INT: now also U3.11 (D4)
- net SNAP_RESET: now also R5.2
- no-connect marks 2 -> 23
Changed lines of the file:
@@
 LIBS:contrib
 LIBS:valves
+LIBS:s1_mini-cache
 EELAYER 25 0
 EELAYER END
@@
 $EndDescr
 $Comp
-L SM220UF1 U?
+L SM220UF1 U2
 U 1 1 57C51AA7
 P 5550 3450
-F 0 "U?" H 5550 5150 60  0000 C CNN
+F 0 "U2" H 5550 5150 60  0000 C CNN
 F 1 "SM220UF1" H 5550 1300 60  0000 C CNN
-F 2 "" H 6250 4700 60  0000 C CNN
+F 2 "CrumpPrints:SM200" H 6250 4700 60  0001 C CNN
 F 3 "" H 6250 4700 60  0000 C CNN
 	1    5550 3450
@@
 $EndComp
 $Comp
-L USB_Edge P?
+L USB_Edge P1
 U 1 1 57C51FF3
 P 3150 2850
-F 0 "P?" H 3400 2650 50  0000 C CNN
+F 0 "P1" H 3400 2650 50  0000 C CNN
 F 1 "USB_Edge" H 3150 3050 50  0000 C CNN
-F 2 "" V 3150 2750 50  0000 C CNN
+F 2 "CrumpPrints:USB_Board_Edge" V 3150 2750 50  0001 C CNN
 F 3 "" V 3150 2750 50  0000 C CNN
 	1    3150 2850
@@
 $EndComp
 $Comp
-L APE8865NL-33-HF-3 U?
-U 1 1 57C522EA
-P 3000 4450
-F 0 "U?" H 2700 4700 50  0000 C CNN
-F 1 "AP2114H-3.3TRG1" H 3000 4650 50  0000 C CNN
-F 2 "SOT-23" H 3000 4550 50  0000 C CIN
-F 3 "" H 3000 4450 50  0000 C CNN
-	1    3000 4450
-	1    0    0    -1
-$EndComp
-$Comp
-L Wemos_D1_Mini U?
+L Wemos_D1_Mini U3
 U 1 1 57C5272C
 P 9050 2500
-F 0 "U?" H 9050 1800 60  0000 C CNN
+F 0 "U3" H 9050 1800 60  0000 C CNN
 F 1 "Wemos_D1_Mini_pins" H 9050 2900 60  0000 C CNN
 F 2 "" H 9050 2500 60  0001 C CNN
@@
 	6300 3000 6350 3000
 $Comp
-L C C?
+L C C1
 U 1 1 57C52C01
 P 2400 4700
-F 0 "C?" H 2425 4800 50  0000 L CNN
+F 0 "C1" H 2425 4800 50  0000 L CNN
 F 1 "C" H 2425 4600 50  0000 L CNN
-F 2 "" H 2438 4550 50  0000 C CNN
+F 2 "Capacitors_SMD:C_0805_HandSoldering" H 2438 4550 50  0001 C CNN
 F 3 "" H 2400 4700 50  0000 C CNN
 	1    2400 4700
@@
 $EndComp
 $Comp
-L C C?
+L C C2
 U 1 1 57C52CCF
 P 3600 4700
-F 0 "C?" H 3625 4800 50  0000 L CNN
+F 0 "C2" H 3625 4800 50  0000 L CNN
 F 1 "C" H 3625 4600 50  0000 L CNN
-F 2 "" H 3638 4550 50  0000 C CNN
+F 2 "Capacitors_SMD:C_0805_HandSoldering" H 3638 4550 50  0001 C CNN
 F 3 "" H 3600 4700 50  0000 C CNN
 	1    3600 4700
@@
 $EndComp
 $Comp
-L GND #PWR?
+L GND #PWR01
 U 1 1 57C52ED6
 P 3000 4950
-F 0 "#PWR?" H 3000 4700 50  0001 C CNN
+F 0 "#PWR01" H 3000 4700 50  0001 C CNN
 F 1 "GND" H 3000 4800 50  0000 C CNN
 F 2 "" H 3000 4950 50  0000 C CNN
@@
 	2400 4950 3600 4950
 Wire Wire Line
-	3000 4950 3000 4750
+	3000 4700 3000 4950
 Wire Wire Line
 	3600 4950 3600 4850
@@
 	2400 4550 2400 4400
 Wire Wire Line
-	2300 4400 2550 4400
+	2300 4400 2600 4400
 Wire Wire Line
 	3600 4550 3600 4400
 Wire Wire Line
-	3450 4400 3700 4400
-$Comp
-L +5V #PWR?
+	3400 4400 3700 4400
+$Comp
+L +5V #PWR02
 U 1 1 57C52F3A
 P 2300 4300
-F 0 "#PWR?" H 2300 4150 50  0001 C CNN
+F 0 "#PWR02" H 2300 4150 50  0001 C CNN
 F 1 "+5V" H 2300 4440 50  0000 C CNN
 F 2 "" H 2300 4300 50  0000 C CNN
@@
 $EndComp
 $Comp
-L +3V3 #PWR?
+L +3V3 #PWR03
 U 1 1 57C52F76
 P 3700 4300
-F 0 "#PWR?" H 3700 4150 50  0001 C CNN
+F 0 "#PWR03" H 3700 4150 50  0001 C CNN
 F 1 "+3V3" H 3700 4440 50  0000 C CNN
 F 2 "" H 3700 4300 50  0000 C CNN
@@
 Connection ~ 3600 4400
 $Comp
-L +5V #PWR?
+L +5V #PWR04
 U 1 1 57C53068
 P 2750 2650
-F 0 "#PWR?" H 2750 2500 50  0001 C CNN
+F 0 "#PWR04" H 2750 2500 50  0001 C CNN
 F 1 "+5V" H 2750 2790 50  0000 C CNN
 F 2 "" H 2750 2650 50  0000 C CNN
@@
 	2750 2700 2750 2650
 $Comp
-L GND #PWR?
+L GND #PWR05
 U 1 1 57C531D5
 P 2750 3050
-F 0 "#PWR?" H 2750 2800 50  0001 C CNN
+F 0 "#PWR05" H 2750 2800 50  0001 C CNN
 F 1 "GND" H 2750 2900 50  0000 C CNN
 F 2 "" H 2750 3050 50  0000 C CNN
@@
 NoConn ~ 2850 2900
 $Comp
-L +3V3 #PWR?
+L +3V3 #PWR06
 U 1 1 57C5338E
 P 4500 2850
-F 0 "#PWR?" H 4500 2700 50  0001 C CNN
+F 0 "#PWR06" H 4500 2700 50  0001 C CNN
 F 1 "+3V3" H 4500 2990 50  0000 C CNN
 F 2 "" H 4500 2850 50  0000 C CNN
@@
 Connection ~ 4750 2000
 $Comp
-L GND #PWR?
+L GND #PWR07
 U 1 1 57C5360C
 P 4550 2250
-F 0 "#PWR?" H 4550 2000 50  0001 C CNN
+F 0 "#PWR07" H 4550 2000 50  0001 C CNN
 F 1 "GND" H 4550 2100 50  0000 C CNN
 F 2 "" H 4550 2250 50  0000 C CNN
@@
 Connection ~ 4750 2200
 Wire Wire Line
-	4750 3600 4800 3600
-Text GLabel 4750 3600 0    60   Input ~ 0
+	4400 3600 4800 3600
+Text GLabel 4400 3600 0    60   Input ~ 0
 SNAP_RESET
 Text GLabel 8450 2300 0    60   Input ~ 0
@@
 	6300 4300 6350 4300
 $Comp
-L R_Small R?
+L R_Small R1
 U 1 1 57C53F16
 P 8950 4450
-F 0 "R?" H 8980 4470 50  0000 L CNN
+F 0 "R1" H 8980 4470 50  0000 L CNN
 F 1 "SR-DR" H 8980 4410 50  0000 L CNN
-F 2 "" H 8950 4450 50  0000 C CNN
+F 2 "Resistors_SMD:R_0805_HandSoldering" H 8950 4450 50  0001 C CNN
 F 3 "" H 8950 4450 50  0000 C CNN
 	1    8950 4450
@@
 $EndComp
 $Comp
-L R_Small R?
+L R_Small R4
 U 1 1 57C53FF5
 P 9400 4900
-F 0 "R?" H 9430 4920 50  0000 L CNN
+F 0 "R4" H 9430 4920 50  0000 L CNN
 F 1 "ST-DT" H 9430 4860 50  0000 L CNN
-F 2 "" H 9400 4900 50  0000 C CNN
+F 2 "Resistors_SMD:R_0805_HandSoldering" H 9400 4900 50  0001 C CNN
 F 3 "" H 9400 4900 50  0000 C CNN
 	1    9400 4900
@@
 $EndComp
 $Comp
-L R_Small R?
+L R_Small R2
 U 1 1 57C54079
 P 8950 4900
-F 0 "R?" H 8980 4920 50  0000 L CNN
+F 0 "R2" H 8980 4920 50  0000 L CNN
 F 1 "SR-DT" H 8980 4860 50  0000 L CNN
-F 2 "" H 8950 4900 50  0000 C CNN
+F 2 "Resistors_SMD:R_0805_HandSoldering" H 8950 4900 50  0001 C CNN
 F 3 "" H 8950 4900 50  0000 C CNN
 	1    8950 4900
@@
 $EndComp
 $Comp
-L R_Small R?
+L R_Small R3
 U 1 1 57C5407F
 P 9400 4450
-F 0 "R?" H 9430 4470 50  0000 L CNN
+F 0 "R3" H 9430 4470 50  0000 L CNN
 F 1 "ST-DR" H 9430 4410 50  0000 L CNN
-F 2 "" H 9400 4450 50  0000 C CNN
+F 2 "Resistors_SMD:R_0805_HandSoldering" H 9400 4450 50  0001 C CNN
 F 3 "" H 9400 4450 50  0000 C CNN
 	1    9400 4450
@@
 	8450 2900 8500 2900
 $Comp
-L +3V3 #PWR?
+L +3V3 #PWR08
 U 1 1 57C55CE8
 P 8450 3100
-F 0 "#PWR?" H 8450 2950 50  0001 C CNN
+F 0 "#PWR08" H 8450 2950 50  0001 C CNN
 F 1 "+3V3" H 8450 3240 50  0000 C CNN
 F 2 "" H 8450 3100 50  0000 C CNN
@@
 $EndComp
 $Comp
-L +5V #PWR?
+L +5V #PWR09
 U 1 1 57C55E11
 P 9650 3100
-F 0 "#PWR?" H 9650 2950 50  0001 C CNN
+F 0 "#PWR09" H 9650 2950 50  0001 C CNN
 F 1 "+5V" H 9650 3240 50  0000 C CNN
 F 2 "" H 9650 3100 50  0000 C CNN
@@
 $EndComp
 $Comp
-L GND #PWR?
+L GND #PWR010
 U 1 1 57C55E21
 P 9900 3100
-F 0 "#PWR?" H 9900 2850 50  0001 C CNN
+F 0 "#PWR010" H 9900 2850 50  0001 C CNN
 F 1 "GND" H 9900 2950 50  0000 C CNN
 F 2 "" H 9900 3100 50  0000 C CNN
@@
 Text Notes 8450 3950 0    60   ~ 0
 SNAP <-> D1 UART Selectors
+$Comp
+L AP2114H U1
+U 1 1 57C56ABD
+P 3000 4450
+F 0 "U1" H 3150 4254 50  0000 C CNN
+F 1 "AP2114H" H 3000 4650 50  0000 C CNN
+F 2 "TO_SOT_Packages_SMD:SOT-223" H 3000 4450 50  0001 C CNN
+F 3 "" H 3000 4450 50  0000 C CNN
+	1    3000 4450
+	1    0    0    -1
+$EndComp
+NoConn ~ 6300 1900
+NoConn ~ 6300 2000
+NoConn ~ 6300 2100
+NoConn ~ 6300 2200
+NoConn ~ 6300 2300
+NoConn ~ 6300 2600
+NoConn ~ 6300 2700
+NoConn ~ 6300 2800
+NoConn ~ 6300 3100
+NoConn ~ 6300 3200
+NoConn ~ 6300 3300
+NoConn ~ 6300 3400
+NoConn ~ 6300 3800
+NoConn ~ 6300 4700
+NoConn ~ 6300 4800
+NoConn ~ 6300 4900
+NoConn ~ 6300 5000
+NoConn ~ 6300 5400
+NoConn ~ 4800 3400
+Wire Wire Line
+	9600 2500 9650 2500
+Wire Wire Line
+	9650 2600 9600 2600
+Wire Wire Line
+	9600 2700 9650 2700
+Wire Wire Line
+	9600 2800 9650 2800
+NoConn ~ 6300 4200
+NoConn ~ 6300 4100
+$Comp
+L R_Small R5
+U 1 1 57C57C90
+P 4550 3400
+F 0 "R5" H 4580 3420 50  0000 L CNN
+F 1 "10K" H 4580 3360 50  0000 L CNN
+F 2 "Resistors_SMD:R_0805_HandSoldering" H 4550 3400 50  0001 C CNN
+F 3 "" H 4550 3400 50  0000 C CNN
+	1    4550 3400
+	1    0    0    -1
+$EndComp
+Wire Wire Line
+	4550 3500 4550 3600
+Connection ~ 4550 3600
+Wire Wire Line
+	4550 3300 4550 3000
+Connection ~ 4550 3000
+$Comp
+L PWR_FLAG #FLG011
+U 1 1 57C589B0
+P 3300 5000
+F 0 "#FLG011" H 3300 5095 50  0001 C CNN
+F 1 "PWR_FLAG" H 3300 5180 50  0000 C CNN
+F 2 "" H 3300 5000 50  0000 C CNN
+F 3 "" H 3300 5000 50  0000 C CNN
+	1    3300 5000
+	-1   0    0    1
+$EndComp
+Wire Wire Line
+	3300 5000 3300 4950
+Connection ~ 3300 4950
 $EndSCHEMATC

Commit message: Add power select resistor.
Parts:
- added R6: 3V3_EN, Resistors_SMD:R_0805_HandSoldering, symbol R_Small
Connections:
- net +3V3: now also R6.1; no longer C2.1, U1.2 (VOUT)
- new net: C2.1, R6.2, U1.2 (VOUT)
Other:
- moved on the sheet: C1, C2, U1
Changed lines of the file:
@@
 L C C1
 U 1 1 57C52C01
-P 2400 4700
-F 0 "C1" H 2425 4800 50  0000 L CNN
-F 1 "C" H 2425 4600 50  0000 L CNN
-F 2 "Capacitors_SMD:C_0805_HandSoldering" H 2438 4550 50  0001 C CNN
-F 3 "" H 2400 4700 50  0000 C CNN
-	1    2400 4700
+P 2400 5000
+F 0 "C1" H 2425 5100 50  0000 L CNN
+F 1 "C" H 2425 4900 50  0000 L CNN
+F 2 "Capacitors_SMD:C_0805_HandSoldering" H 2438 4850 50  0001 C CNN
+F 3 "" H 2400 5000 50  0000 C CNN
+	1    2400 5000
 	1    0    0    -1
 $EndComp
@@
 L C C2
 U 1 1 57C52CCF
-P 3600 4700
-F 0 "C2" H 3625 4800 50  0000 L CNN
-F 1 "C" H 3625 4600 50  0000 L CNN
-F 2 "Capacitors_SMD:C_0805_HandSoldering" H 3638 4550 50  0001 C CNN
-F 3 "" H 3600 4700 50  0000 C CNN
-	1    3600 4700
+P 3600 5000
+F 0 "C2" H 3625 5100 50  0000 L CNN
+F 1 "C" H 3625 4900 50  0000 L CNN
+F 2 "Capacitors_SMD:C_0805_HandSoldering" H 3638 4850 50  0001 C CNN
+F 3 "" H 3600 5000 50  0000 C CNN
+	1    3600 5000
 	1    0    0    -1
 $EndComp
@@
 L GND #PWR01
 U 1 1 57C52ED6
-P 3000 4950
-F 0 "#PWR01" H 3000 4700 50  0001 C CNN
-F 1 "GND" H 3000 4800 50  0000 C CNN
-F 2 "" H 3000 4950 50  0000 C CNN
-F 3 "" H 3000 4950 50  0000 C CNN
-	1    3000 4950
-	1    0    0    -1
-$EndComp
-Wire Wire Line
-	2400 4850 2400 4950
-Wire Wire Line
-	2400 4950 3600 4950
-Wire Wire Line
-	3000 4700 3000 4950
-Wire Wire Line
-	3600 4950 3600 4850
-Connection ~ 3000 4950
-Wire Wire Line
-	2400 4550 2400 4400
-Wire Wire Line
-	2300 4400 2600 4400
-Wire Wire Line
-	3600 4550 3600 4400
-Wire Wire Line
-	3400 4400 3700 4400
+P 3000 5250
+F 0 "#PWR01" H 3000 5000 50  0001 C CNN
+F 1 "GND" H 3000 5100 50  0000 C CNN
+F 2 "" H 3000 5250 50  0000 C CNN
+F 3 "" H 3000 5250 50  0000 C CNN
+	1    3000 5250
+	1    0    0    -1
+$EndComp
+Wire Wire Line
+	2400 5150 2400 5250
+Wire Wire Line
+	2400 5250 3600 5250
+Wire Wire Line
+	3000 5000 3000 5250
+Wire Wire Line
+	3600 5250 3600 5150
+Connection ~ 3000 5250
+Wire Wire Line
+	2400 4850 2400 4700
+Wire Wire Line
+	2300 4700 2600 4700
+Wire Wire Line
+	3600 4850 3600 4700
+Wire Wire Line
+	3700 4700 3400 4700
 $Comp
 L +5V #PWR02
 U 1 1 57C52F3A
-P 2300 4300
-F 0 "#PWR02" H 2300 4150 50  0001 C CNN
-F 1 "+5V" H 2300 4440 50  0000 C CNN
-F 2 "" H 2300 4300 50  0000 C CNN
-F 3 "" H 2300 4300 50  0000 C CNN
-	1    2300 4300
+P 2300 4600
+F 0 "#PWR02" H 2300 4450 50  0001 C CNN
+F 1 "+5V" H 2300 4740 50  0000 C CNN
+F 2 "" H 2300 4600 50  0000 C CNN
+F 3 "" H 2300 4600 50  0000 C CNN
+	1    2300 4600
 	1    0    0    -1
 $EndComp
@@
 $EndComp
 Wire Wire Line
-	2300 4300 2300 4400
-Connection ~ 2400 4400
-Wire Wire Line
-	3700 4400 3700 4300
-Connection ~ 3600 4400
+	2300 4600 2300 4700
+Connection ~ 2400 4700
+Wire Wire Line
+	3700 4550 3700 4700
+Connection ~ 3600 4700
 $Comp
 L +5V #PWR04
@@
 L AP2114H U1
 U 1 1 57C56ABD
-P 3000 4450
-F 0 "U1" H 3150 4254 50  0000 C CNN
-F 1 "AP2114H" H 3000 4650 50  0000 C CNN
-F 2 "TO_SOT_Packages_SMD:SOT-223" H 3000 4450 50  0001 C CNN
-F 3 "" H 3000 4450 50  0000 C CNN
-	1    3000 4450
+P 3000 4750
+F 0 "U1" H 3150 4554 50  0000 C CNN
+F 1 "AP2114H" H 3000 4950 50  0000 C CNN
+F 2 "TO_SOT_Packages_SMD:SOT-223" H 3000 4750 50  0001 C CNN
+F 3 "" H 3000 4750 50  0000 C CNN
+	1    3000 4750
 	1    0    0    -1
 $EndComp
@@
 L PWR_FLAG #FLG011
 U 1 1 57C589B0
-P 3300 5000
-F 0 "#FLG011" H 3300 5095 50  0001 C CNN
-F 1 "PWR_FLAG" H 3300 5180 50  0000 C CNN
-F 2 "" H 3300 5000 50  0000 C CNN
-F 3 "" H 3300 5000 50  0000 C CNN
-	1    3300 5000
+P 3300 5300
+F 0 "#FLG011" H 3300 5395 50  0001 C CNN
+F 1 "PWR_FLAG" H 3300 5480 50  0000 C CNN
+F 2 "" H 3300 5300 50  0000 C CNN
+F 3 "" H 3300 5300 50  0000 C CNN
+	1    3300 5300
 	-1   0    0    1
 $EndComp
 Wire Wire Line
-	3300 5000 3300 4950
-Connection ~ 3300 4950
+	3300 5300 3300 5250
+Connection ~ 3300 5250
+$Comp
+L R_Small R6
+U 1 1 57C62FB9
+P 3700 4450
+F 0 "R6" H 3730 4470 50  0000 L CNN
+F 1 "3V3_EN" H 3730 4410 50  0000 L CNN
+F 2 "Resistors_SMD:R_0805_HandSoldering" H 3700 4450 50  0001 C CNN
+F 3 "" H 3700 4450 50  0000 C CNN
+	1    3700 4450
+	1    0    0    -1
+$EndComp
+Wire Wire Line
+	3700 4350 3700 4300
+$Comp
+L PWR_FLAG #FLG012
+U 1 1 57C63CE4
+P 8650 3250
+F 0 "#FLG012" H 8650 3345 50  0001 C CNN
+F 1 "PWR_FLAG" H 8650 3430 50  0000 C CNN
+F 2 "" H 8650 3250 50  0000 C CNN
+F 3 "" H 8650 3250 50  0000 C CNN
+	1    8650 3250
+	-1   0    0    1
+$EndComp
+Wire Wire Line
+	8650 3250 8650 3050
+Wire Wire Line
+	8650 3050 8450 3050
+Connection ~ 8450 3050
 $EndSCHEMATC

Commit message: Place parts.
Parts:
- U3: value Wemos_D1_Mini_pins -> Wemos_D1_Mini; footprint (none) -> CrumpPrints:D1_mini
Changed lines of the file:
@@
 EESchema Schematic File Version 2
+LIBS:s1_mini-rescue
 LIBS:crumpschemes
 LIBS:power
@@
 	0    1    1    0
 $EndComp
-$Comp
-L Wemos_D1_Mini U3
-U 1 1 57C5272C
-P 9050 2500
-F 0 "U3" H 9050 1800 60  0000 C CNN
-F 1 "Wemos_D1_Mini_pins" H 9050 2900 60  0000 C CNN
-F 2 "" H 9050 2500 60  0001 C CNN
-F 3 "" H 9050 2500 60  0001 C CNN
-	1    9050 2500
-	1    0    0    -1
-$EndComp
 Text GLabel 6350 2900 2    60   Input ~ 0
 SNAP_RXD1
@@
 $EndComp
 $Comp
-L GND #PWR01
+L GND #PWR4
 U 1 1 57C52ED6
 P 3000 5250
-F 0 "#PWR01" H 3000 5000 50  0001 C CNN
+F 0 "#PWR4" H 3000 5000 50  0001 C CNN
 F 1 "GND" H 3000 5100 50  0000 C CNN
 F 2 "" H 3000 5250 50  0000 C CNN
@@
 	3700 4700 3400 4700
 $Comp
-L +5V #PWR02
+L +5V #PWR1
 U 1 1 57C52F3A
 P 2300 4600
-F 0 "#PWR02" H 2300 4450 50  0001 C CNN
+F 0 "#PWR1" H 2300 4450 50  0001 C CNN
 F 1 "+5V" H 2300 4740 50  0000 C CNN
 F 2 "" H 2300 4600 50  0000 C CNN
@@
 $EndComp
 $Comp
-L +3V3 #PWR03
+L +3V3 #PWR5
 U 1 1 57C52F76
 P 3700 4300
-F 0 "#PWR03" H 3700 4150 50  0001 C CNN
+F 0 "#PWR5" H 3700 4150 50  0001 C CNN
 F 1 "+3V3" H 3700 4440 50  0000 C CNN
 F 2 "" H 3700 4300 50  0000 C CNN
@@
 Connection ~ 3600 4700
 $Comp
-L +5V #PWR04
+L +5V #PWR2
 U 1 1 57C53068
 P 2750 2650
-F 0 "#PWR04" H 2750 2500 50  0001 C CNN
+F 0 "#PWR2" H 2750 2500 50  0001 C CNN
 F 1 "+5V" H 2750 2790 50  0000 C CNN
 F 2 "" H 2750 2650 50  0000 C CNN
@@
 	2750 2700 2750 2650
 $Comp
-L GND #PWR05
+L GND #PWR3
 U 1 1 57C531D5
 P 2750 3050
-F 0 "#PWR05" H 2750 2800 50  0001 C CNN
+F 0 "#PWR3" H 2750 2800 50  0001 C CNN
 F 1 "GND" H 2750 2900 50  0000 C CNN
 F 2 "" H 2750 3050 50  0000 C CNN
@@
 NoConn ~ 2850 2900
 $Comp
-L +3V3 #PWR06
+L +3V3 #PWR6
 U 1 1 57C5338E
 P 4500 2850
-F 0 "#PWR06" H 4500 2700 50  0001 C CNN
+F 0 "#PWR6" H 4500 2700 50  0001 C CNN
 F 1 "+3V3" H 4500 2990 50  0000 C CNN
 F 2 "" H 4500 2850 50  0000 C CNN
@@
 Connection ~ 4750 2000
 $Comp
-L GND #PWR07
+L GND #PWR7
 U 1 1 57C5360C
 P 4550 2250
-F 0 "#PWR07" H 4550 2000 50  0001 C CNN
+F 0 "#PWR7" H 4550 2000 50  0001 C CNN
 F 1 "GND" H 4550 2100 50  0000 C CNN
 F 2 "" H 4550 2250 50  0000 C CNN
@@
 	8450 2900 8500 2900
 $Comp
-L +3V3 #PWR08
+L +3V3 #PWR8
 U 1 1 57C55CE8
 P 8450 3100
-F 0 "#PWR08" H 8450 2950 50  0001 C CNN
+F 0 "#PWR8" H 8450 2950 50  0001 C CNN
 F 1 "+3V3" H 8450 3240 50  0000 C CNN
 F 2 "" H 8450 3100 50  0000 C CNN
@@
 $EndComp
 $Comp
-L +5V #PWR09
+L +5V #PWR9
 U 1 1 57C55E11
 P 9650 3100
-F 0 "#PWR09" H 9650 2950 50  0001 C CNN
+F 0 "#PWR9" H 9650 2950 50  0001 C CNN
 F 1 "+5V" H 9650 3240 50  0000 C CNN
 F 2 "" H 9650 3100 50  0000 C CNN
@@
 $EndComp
 $Comp
-L GND #PWR010
+L GND #PWR10
 U 1 1 57C55E21
 P 9900 3100
-F 0 "#PWR010" H 9900 2850 50  0001 C CNN
+F 0 "#PWR10" H 9900 2850 50  0001 C CNN
 F 1 "GND" H 9900 2950 50  0000 C CNN
 F 2 "" H 9900 3100 50  0000 C CNN
@@
 Connection ~ 4550 3000
 $Comp
-L PWR_FLAG #FLG011
+L PWR_FLAG #FLG1
 U 1 1 57C589B0
 P 3300 5300
-F 0 "#FLG011" H 3300 5395 50  0001 C CNN
+F 0 "#FLG1" H 3300 5395 50  0001 C CNN
 F 1 "PWR_FLAG" H 3300 5480 50  0000 C CNN
 F 2 "" H 3300 5300 50  0000 C CNN
@@
 	3700 4350 3700 4300
 $Comp
-L PWR_FLAG #FLG012
+L PWR_FLAG #FLG2
 U 1 1 57C63CE4
 P 8650 3250
-F 0 "#FLG012" H 8650 3345 50  0001 C CNN
+F 0 "#FLG2" H 8650 3345 50  0001 C CNN
 F 1 "PWR_FLAG" H 8650 3430 50  0000 C CNN
 F 2 "" H 8650 3250 50  0000 C CNN
@@
 	8650 3050 8450 3050
 Connection ~ 8450 3050
+$Comp
+L Wemos_D1_Mini U3
+U 1 1 57C63B2C
+P 9050 2500
+F 0 "U3" H 9050 1800 60  0000 C CNN
+F 1 "Wemos_D1_Mini" H 9050 2900 60  0000 C CNN
+F 2 "CrumpPrints:D1_mini" H 9050 2500 60  0001 C CNN
+F 3 "" H 9050 2500 60  0001 C CNN
+	1    9050 2500
+	1    0    0    -1
+$EndComp
 $EndSCHEMATC
